File: painel_pcb2/painel_pcb2.kicad_pcb (KiCad board)
At the start: 2 copper layers, 91.4 x 119.4 mm, 53 parts, among them J1 Conn_02x16_Counter_Clockwise, J2 Conn_02x02_Counter_Clockwise, J3 Conn_02x06_Counter_Clockwise, J4 Conn_02x08_Counter_Clockwise, J5 Conn_02x03_Counter_Clockwise, U1 MAX7219, U2 MAX7219, U3 74LS595

Commit message: converted to KICAD 6
Connections:
- net ~RESET renamed ~{RESET}
Other:
- net class Default removed
