File: painel_pcb1/painel_pcb1.kicad_pcb (KiCad board)
At the start: 2 copper layers, 91.4 x 119.4 mm, 57 parts, among them J1 Conn_02x16_Counter_Clockwise, J2 Conn_02x02_Counter_Clockwise, J3 Conn_02x06_Counter_Clockwise, J4 Conn_02x08_Counter_Clockwise, J5 Conn_02x03_Counter_Clockwise, J6 Conn_02x08_Counter_Clockwise, U1 MAX7219, U2 MAX7219, U3 74LS595, U4 74LS595

Commit message: converted to KICAD 6
Connections:
- net ~RESET renamed ~{RESET}
Other:
- net class Default removed

Commit message: wip
Parts:
- added U5: Pico, MCU_RaspberryPi_and_Boards:RPi_Pico_SMD_TH, B.Cu at (114.3, 119.4)
Connections:
- A1 pad 1: Net-(A1-Pad1) -> unconnected-(A1-Pad1)

Commit message: wip
Parts:
- added J7: Conn_02x18_Counter_Clockwise, Connector_PinHeader_2.54mm:PinHeader_2x18_P2.54mm_Vertical, B.Cu at (71.1, 149.9)
- J6: moved to B.Cu
- moved J2 8.89 mm to (55.9, 129.5)
- moved J1 7.73 mm to (71.1, 142.2)
- moved J6 2.84 mm to (139.7, 55.9), turned to 180 degrees
- moved J5 1.27 mm to (137.2, 151.1)
Connections:
- A1 pad 19: CLOCK -> GPIO2
- A1 pad 4: +3V3 -> 3V3
- A1 pad 5: +5V -> VBUS
- C1 pad 1: +5V -> VBUS
- C2 pad 1: +5V -> VBUS
- C3 pad 1: +5V -> VBUS
- C4 pad 1: +5V -> VBUS
- C5 pad 1: +5V -> VBUS
- C6 pad 1: +5V -> VBUS
- J1 pad 31: +3V3 -> 3V3
- J1 pad 32: +5V -> VBUS
- J1 pad 5: CLOCK -> GPIO2
- J5 pad 1: +5V -> VBUS
- J5 pad 2: +3V3 -> 3V3
- J5 pad 5: CLOCK -> GPIO2
- R1 pad 1: +5V -> VBUS
- R2 pad 1: +5V -> VBUS
- U1 pad 13: CLOCK -> GPIO2
- U1 pad 19: +5V -> VBUS
- U2 pad 13: CLOCK -> GPIO2
- U2 pad 19: +5V -> VBUS
- U3 pad 10: +5V -> VBUS
- U3 pad 11: CLOCK -> GPIO2
- U3 pad 16: +5V -> VBUS
- U4 pad 10: +5V -> VBUS
- U4 pad 11: CLOCK -> GPIO2
- U4 pad 16: +5V -> VBUS
- U5 pad 1: unconnected-(U5-Pad1) -> GPIO0
- U5 pad 10: unconnected-(U5-Pad10) -> GPIO7
- U5 pad 11: unconnected-(U5-Pad11) -> GPIO8
- U5 pad 12: unconnected-(U5-Pad12) -> GPIO9
- U5 pad 13: unconnected-(U5-Pad13) -> GND
- U5 pad 14: unconnected-(U5-Pad14) -> GPIO10
- U5 pad 15: unconnected-(U5-Pad15) -> GPIO11
- U5 pad 16: unconnected-(U5-Pad16) -> GPIO12
- U5 pad 17: unconnected-(U5-Pad17) -> GPIO13
- U5 pad 18: unconnected-(U5-Pad18) -> GND
- U5 pad 19: unconnected-(U5-Pad19) -> GPIO14
- U5 pad 2: unconnected-(U5-Pad2) -> GPIO1
- U5 pad 20: unconnected-(U5-Pad20) -> GPIO15
- U5 pad 21: unconnected-(U5-Pad21) -> GPIO16
- U5 pad 22: unconnected-(U5-Pad22) -> GPIO17
- U5 pad 23: unconnected-(U5-Pad23) -> GND
- U5 pad 24: unconnected-(U5-Pad24) -> GPIO18
- U5 pad 25: unconnected-(U5-Pad25) -> GPIO19
- U5 pad 26: unconnected-(U5-Pad26) -> GPIO20
- U5 pad 27: unconnected-(U5-Pad27) -> GPIO21
- U5 pad 28: unconnected-(U5-Pad28) -> GND
- U5 pad 29: unconnected-(U5-Pad29) -> GPIO22
- U5 pad 3: unconnected-(U5-Pad3) -> GND
- U5 pad 30: unconnected-(U5-Pad30) -> RUN
- U5 pad 31: unconnected-(U5-Pad31) -> GPIO26
- U5 pad 32: unconnected-(U5-Pad32) -> GPIO27
- U5 pad 33: unconnected-(U5-Pad33) -> GND
- U5 pad 34: unconnected-(U5-Pad34) -> GPIO28
- U5 pad 35: unconnected-(U5-Pad35) -> ADC_VREF
- U5 pad 36: unconnected-(U5-Pad36) -> 3V3
- U5 pad 37: unconnected-(U5-Pad37) -> 3V3_EN
- U5 pad 38: unconnected-(U5-Pad38) -> GND
- U5 pad 39: unconnected-(U5-Pad39) -> VSYS
- U5 pad 4: unconnected-(U5-Pad4) -> GPIO2
- U5 pad 40: unconnected-(U5-Pad40) -> VBUS
- U5 pad 42: unconnected-(U5-Pad42) -> GND
- U5 pad 5: unconnected-(U5-Pad5) -> D2
- U5 pad 6: unconnected-(U5-Pad6) -> GPIO4
- U5 pad 7: unconnected-(U5-Pad7) -> D3
- U5 pad 8: unconnected-(U5-Pad8) -> GND
- U5 pad 9: unconnected-(U5-Pad9) -> GPIO6

Commit message: autorouting
Parts:
- removed A1: Arduino_UNO_R3, Module:Arduino_UNO_R3
- added J8: Conn_01x06, Connector_PinHeader_2.54mm:PinHeader_1x06_P2.54mm_Vertical, B.Cu at (56.0, 138.5)
- J1: value Conn_02x16_Counter_Clockwise -> Conn_01x04; footprint Connector_PinHeader_2.54mm:PinHeader_2x16_P2.54mm_Vertical -> Connector_PinHeader_2.54mm:PinHeader_1x04_P2.54mm_Vertical
- moved C5 57.1 mm to (116.9, 93.8)
- moved U4 57.1 mm to (120.8, 88.7)
- moved C6 24.0 mm to (87.7, 94.1)
- moved U3 24.0 mm to (91.5, 89.0)
- moved J1 11.2 mm to (60.6, 138.5), turned to 180 degrees
- moved C1 7.13 mm to (113.9, 59.1)
- moved C2 7.13 mm to (121.6, 57.9)
- moved R1 7.13 mm to (100.0, 59.1)
- moved U2 7.13 mm to (100.0, 62.9)
- moved U1 5.98 mm to (65.9, 63.0)
- moved C4 5.98 mm to (86.2, 57.9)
- moved C3 5.98 mm to (79.9, 59.1)
- moved R2 5.98 mm to (65.9, 59.1)
- moved J7 5.58 mm to (69.6, 144.5)
- moved J4 2.35 mm to (55.5, 74.1)
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Connections:
- J1 pad 1: D0 -> GPIO6
- J1 pad 2: D1 -> GPIO7
- J1 pad 3: D2 -> GPIO8
- J1 pad 4: D3 -> GPIO9
- J5 pad 4: D3 -> GPIO5
- J5 pad 5: GPIO2 -> CLOCK
- J7 pad 3: GPIO2 -> CLOCK
- J7 pad 4: D2 -> DATA
- J7 pad 6: D3 -> GPIO5
- U1 pad 1: D2 -> DATA
- U1 pad 12: D3 -> GPIO5
- U1 pad 13: GPIO2 -> CLOCK
- U2 pad 12: D3 -> GPIO5
- U2 pad 13: GPIO2 -> CLOCK
- U3 pad 11: GPIO2 -> CLOCK
- U3 pad 12: D3 -> GPIO5
- U4 pad 11: GPIO2 -> CLOCK
- U4 pad 12: D3 -> GPIO5
- U5 pad 4: GPIO2 -> CLOCK
- U5 pad 5: D2 -> DATA
- U5 pad 7: D3 -> GPIO5
Routing:
- net GND: track 0.00 -> 408.5 mm
- net GPIO5: track 0.00 -> 339.6 mm, vias 0 -> 1
- net SEG_1_D: track 0.00 -> 310.3 mm, vias 0 -> 2
- net SEG_1_G: track 0.00 -> 297.5 mm, vias 0 -> 2
- net VBUS: track 0.00 -> 277.5 mm
- net SEG_1_C: track 0.00 -> 276.8 mm, vias 0 -> 1
- net SEG_1_A: track 0.00 -> 262.2 mm, vias 0 -> 2
- net SEG_1_F: track 0.00 -> 254.9 mm, vias 0 -> 3
- net CLOCK: track 0.00 -> 245.6 mm
- net SEG_1_B: track 0.00 -> 238.2 mm, vias 0 -> 1
- net SEG_1_E: track 0.00 -> 234.3 mm
- net DIG_1_4: track 0.00 -> 225.9 mm
- net SEG_1_DP: track 0.00 -> 224.5 mm, vias 0 -> 1
- net DIG_1_3: track 0.00 -> 181.8 mm, vias 0 -> 1
- net DATA: track 0.00 -> 157.8 mm
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
Commit message: Eu acho que essa versão da PCB tá quase boa pra mandar rodar
Parts:
- added H1: MountingHole, MountingHole:MountingHole_3.2mm_M3, F.Cu at (136.9, 140.5)
- added H2: MountingHole, MountingHole:MountingHole_3.2mm_M3, F.Cu at (55.5, 142.3)
- added H3: MountingHole, MountingHole:MountingHole_3.2mm_M3, F.Cu at (66.9, 55.1)
- added H4: MountingHole, MountingHole:MountingHole_3.2mm_M3, F.Cu at (128.4, 55.1)
- moved J7 10.9 mm to (80.5, 145.4)
- moved J8 10.6 mm to (57.6, 149.0), turned to -90 degrees
- moved J1 5.84 mm to (62.8, 144.0), turned to -90 degrees
- moved J2 3.27 mm to (58.1, 131.9)
- moved U2 3.04 mm to (100.0, 66.0)
- moved C1 3.04 mm to (114.0, 62.2)
- moved C2 3.04 mm to (121.6, 60.9)
- moved C3 3.04 mm to (79.9, 62.2)
- moved C4 3.04 mm to (86.3, 60.9)
- moved R1 3.04 mm to (100.0, 62.2)
- moved R2 3.04 mm to (66.0, 62.2)
- moved U1 3.04 mm to (66.0, 66.0)
- moved U5 1.75 mm to (116.0, 119.9)
Routing:
- net GPIO5: track 339.6 -> 235.7 mm
- net SEG_1_G: track 297.5 -> 242.0 mm, vias 2 -> 1
- net CLOCK: track 245.6 -> 204.8 mm, vias 0 -> 1
- net SEG_1_F: track 254.9 -> 224.2 mm, vias 3 -> 0
- net SEG_1_B: track 238.2 -> 263.5 mm, vias 1 -> 0
- net GPIO22: track 58.8 -> 34.9 mm, vias 1 -> 0
- net DOUT_7: track 60.4 -> 82.6 mm
- net SEG_2_G: track 99.8 -> 78.2 mm, vias 0 -> 1
- net SEG_1_A: track 262.2 -> 280.5 mm, vias 2 -> 1
- net DATA: track 157.8 -> 175.7 mm, vias 0 -> 1
- net SEG_2_C: track 85.5 -> 68.0 mm, vias 0 -> 1
- net 3V3: track 72.8 -> 56.5 mm
- net DIG_2_3: track 78.5 -> 63.9 mm
- net DIG_1_4: track 225.9 -> 240.2 mm
- net GPIO9: track 80.5 -> 66.2 mm
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Other:
- board text added: "74LS595"
- board text added: "Chaves & Botões"
- board text added: "Colunas"
- board text added: "Em comemoração aos 50 anos da inauguração do computador Patinho Feio da Escola Politécnica da Universidade de São Paulo."
- board text added: "LED TRANSBORDO"
- board text added: "LED VAI-UM"
- board text added: "LEDS - DADOS DO PAINEL"
- board text added: "LEDS - ENDEREÇO DE INSTRUÇÃO"
- board text added: "LEDS - ENDEREÇO NA MEMÓRIA"
- board text added: "Linhas"
- board text added: "MAX7219"
- board text added: "Raspberry Pi Pico"
- board text added: "Saída paralela"
- board text added: "Setembro/2022 Felipe {dblquote}Juca{dblquote} Sanches juca@members.fsf.org https://forum.fiozera.com.br/t/resgate-historico-do-computador-patinho-feio-usp-1971"
- board text added: "Sinais do RPi-Pico"
- board text added: "Sinais para extensão com shift-registers"
- board text added: "https://github.com/ArqueologiaDigital/PatinhoFeio_Painel_KICAD"
